Commit message: Update .urdf

File: ros/src/troggie_description/urdf/troggie.urdf.xacro (robot description, xacro)
@@ -21,7 +21,7 @@
     </visual>
     <collision>
-      <origin xyz="${troggie_bumper_extend / 200.0} 0 ${base_z_size/4}" rpy="0 0 0" />
+      <origin xyz="${20 / 200.0} 0 ${base_z_size/4}" rpy="0 0 0" />
       <geometry>
-        <box size="${base_x_size + troggie_bumper_extend / 100.0} ${base_y_size} ${base_z_size/2}"/>
+        <box size="${base_x_size + 20 / 100.0} ${base_y_size} ${base_z_size/2}"/>
       </geometry>
     </collision>

Commit message: Testing drive controller

File: ros/src/troggie_description/urdf/troggie.urdf.xacro (robot description, xacro)
@@ -14,5 +14,5 @@
   <!-- Wheel Properties -->
   <xacro:property name="wheel_length" value="0.1143" />
-  <xacro:property name="wheel_radius" value="0.1651" />
+  <xacro:property name="wheel_radius" value="0.5" />
   <xacro:include filename="$(find troggie_description)/urdf/wheel.urdf.xacro" />
   <!-- Base link is the center of the robot's bottom plate -->

Commit message: Set wheel radius parameter

File: ros/src/troggie_description/urdf/troggie.urdf.xacro (robot description, xacro)
@@ -14,5 +14,5 @@
   <!-- Wheel Properties -->
   <xacro:property name="wheel_length" value="0.1143" />
-  <xacro:property name="wheel_radius" value="0.5" />
+  <xacro:property name="wheel_radius" value="0.127" />
   <xacro:include filename="$(find troggie_description)/urdf/wheel.urdf.xacro" />
   <!-- Base link is the center of the robot's bottom plate -->
