Commit message: Remove troggie

File: ros/src/trog_description/urdf/troggie.urdf.xacro (robot description, xacro)
@@ -1,4 +1,4 @@
 <?xml version="1.0"?>
-<robot name="troggie" xmlns:xacro="http://ros.org/wiki/xacro">
+<robot name="trog" xmlns:xacro="http://ros.org/wiki/xacro">
   <xacro:arg name="robot_namespace" default="/" />
   <xacro:arg name="urdf_extras" default="empty.urdf" />
@@ -15,5 +15,5 @@
   <xacro:property name="wheel_length" value="0.1143" />
   <xacro:property name="wheel_radius" value="0.127" />
-  <xacro:include filename="$(find troggie_description)/urdf/wheel.urdf.xacro" />
+  <xacro:include filename="$(find trog_description)/urdf/wheel.urdf.xacro" />
   <!-- Base link is the center of the robot's bottom plate -->
   <link name="base_link">
@@ -65,16 +65,16 @@
   </gazebo>
   <!-- Husky wheel macros -->
-  <xacro:troggie_wheel wheel_prefix="front_left">
+  <xacro:trog_wheel wheel_prefix="front_left">
     <origin xyz="${wheelbase/2} ${track/2} ${wheel_vertical_offset}" rpy="0 0 0" />
-  </xacro:troggie_wheel>
-  <xacro:troggie_wheel wheel_prefix="front_right">
+  </xacro:trog_wheel>
+  <xacro:trog_wheel wheel_prefix="front_right">
     <origin xyz="${wheelbase/2} ${-track/2} ${wheel_vertical_offset}" rpy="0 0 0" />
-  </xacro:troggie_wheel>
-  <xacro:troggie_wheel wheel_prefix="rear_left">
+  </xacro:trog_wheel>
+  <xacro:trog_wheel wheel_prefix="rear_left">
     <origin xyz="${-wheelbase/2} ${track/2} ${wheel_vertical_offset}" rpy="0 0 0" />
-  </xacro:troggie_wheel>
-  <xacro:troggie_wheel wheel_prefix="rear_right">
+  </xacro:trog_wheel>
+  <xacro:trog_wheel wheel_prefix="rear_right">
     <origin xyz="${-wheelbase/2} ${-track/2} ${wheel_vertical_offset}" rpy="0 0 0" />
-  </xacro:troggie_wheel>
+  </xacro:trog_wheel>
   <!-- <xacro:if value="$(arg laser_enabled)">
     <sick_lms1xx_mount prefix="base"/>

File: ros/src/trog_description/urdf/wheel.urdf.xacro (robot description, xacro)
@@ -21,6 +21,6 @@
 ARISING IN ANY WAY OUT OF THE USE OF THIS SOFTWARE, EVEN IF ADVISED OF THE POSSIBILITY OF SUCH DAMAGE.
 -->
-<robot xmlns:xacro="http://ros.org/wiki/xacro" name="troggie_wheel">
-	<xacro:macro name="troggie_wheel" params="wheel_prefix *joint_pose">
+<robot xmlns:xacro="http://ros.org/wiki/xacro" name="trog_wheel">
+	<xacro:macro name="trog_wheel" params="wheel_prefix *joint_pose">
 		<link name="${wheel_prefix}_wheel_link">
 			<inertial>
@@ -32,5 +32,5 @@
 				<origin xyz="0 0 0" rpy="0 0 0" />
 				<geometry>
-					<mesh filename="package://troggie_description/meshes/wheel.dae" />
+					<mesh filename="package://trog_description/meshes/wheel.dae" />
 				</geometry>
 			</visual>

Commit message: Configure troggie.urdf.xacro

File: ros/src/trog_description/urdf/troggie.urdf.xacro (robot description, xacro)
@@ -5,13 +5,13 @@
   <xacro:property name="M_PI" value="3.14159"/>
   <!-- Base Size -->
-  <xacro:property name="base_x_size" value="0.98740000" />
-  <xacro:property name="base_y_size" value="0.57090000" />
-  <xacro:property name="base_z_size" value="0.24750000" />
+  <xacro:property name="base_x_size" value="0.48260000" />
+  <xacro:property name="base_y_size" value="0.35560000" />
+  <xacro:property name="base_z_size" value="0.49530000" />
   <!-- Wheel Mounting Positions -->
-  <xacro:property name="wheelbase" value="0.5120" />
-  <xacro:property name="track" value="0.5708" />
-  <xacro:property name="wheel_vertical_offset" value="0.03282" />
+  <xacro:property name="wheelbase" value="0.4064" />
+  <xacro:property name="track" value="0.4826" />
+  <xacro:property name="wheel_vertical_offset" value="0.127" />
   <!-- Wheel Properties -->
-  <xacro:property name="wheel_length" value="0.1143" />
+  <xacro:property name="wheel_length" value="0.0762" />
   <xacro:property name="wheel_radius" value="0.127" />
   <xacro:include filename="$(find trog_description)/urdf/wheel.urdf.xacro" />
@@ -42,5 +42,5 @@
   </joint>
   <!-- Interial link stores the robot's inertial information -->
-  <link name="inertial_link">
+  <!-- <link name="inertial_link">
     <inertial>
       <mass value="46.034" />
@@ -48,13 +48,13 @@
       <inertia ixx="0.6022" ixy="-0.02364" ixz="-0.1197" iyy="1.7386" iyz="-0.001544" izz="2.0296" />
     </inertial>
-  </link>
-  <joint name="inertial_joint" type="fixed">
+  </link> -->
+  <!-- <joint name="inertial_joint" type="fixed">
     <origin xyz="0 0 0" rpy="0 0 0" />
     <parent link="base_link" />
     <child link="inertial_link" />
-  </joint>
+  </joint> -->
   <!-- IMU Link is the standard mounting position for the UM6 IMU.-->
   <!-- Can be modified with environment variables in /etc/ros/setup.bash -->
-  <link name="imu_link"/>
+  <!-- <link name="imu_link"/>
   <joint name="imu_joint" type="fixed">
     <origin xyz="$(optenv HUSKY_IMU_XYZ 0.19 0 0.149)" rpy="$(optenv HUSKY_IMU_RPY 0 -1.5708 3.1416)" />
@@ -63,5 +63,5 @@
   </joint>
   <gazebo reference="imu_link">
-  </gazebo>
+  </gazebo> -->
   <!-- Husky wheel macros -->
   <xacro:trog_wheel wheel_prefix="front_left">
